File: kicad/mcu/mcu.kicad_sch (KiCad schematic)
At the start: 23 parts, among them J1 Conn_01x05, J2 Conn_01x04, Q1 BC817, U1 AMS1117-3.3, U2 STM32F030F4Px

Commit message: Поробуем на плате разместить eeprom
Parts:
- removed U1: AMS1117-3.3, Package_TO_SOT_SMD:SOT-223-3_TabPin2, symbol Regulator_Linear:AMS1117-3.3
- added C4, C5: 0.1, Capacitor_SMD:C_1206_3216Metric, symbol Device:C
- added C6: 100.0x6.3V, Capacitor_Tantalum_SMD:CP_EIA-3528-21_Kemet-B_Pad1.50x2.35mm_HandSolder, symbol Device:C_Polarized
- added R11: 64, Resistor_SMD:R_1206_3216Metric, symbol Device:R
- added U1: LM1117-3.3, Package_TO_SOT_SMD:SOT-223, symbol Regulator_Linear:LM1117-3.3
- added U3: AT24CS64-SSHM, Package_SO:SO-8_5.3x6.2mm_P1.27mm, symbol Memory_EEPROM:AT24CS64-SSHM
- C2: value C -> 0.1
- C3: value C_Polarized -> 100.0x6.3V; footprint Capacitor_SMD:C_1210_3225Metric -> Capacitor_Tantalum_SMD:CP_EIA-3528-21_Kemet-B_Pad1.50x2.35mm_HandSolder
- Q1: Цена (none) -> 4
- R10: value 224 -> 1k
- U2: value STM32F030F4Px -> STM32F030F4P6; Цена (none) -> 100
Connections:
- net +3.3V: now also C5.1, U1.2 (VO), U3.8 (VCC)
- net GNDD: now also C4.2, C5.2, C6.2, U1.1 (GND), U3.1 (A0), U3.2 (A1), U3.3 (A2), U3.4 (GND), U3.7 (WP); no longer D1.4 (BA)
- net LED2_1: now also R6.1, U2.6 (PA0); no longer R4.1, U2.14 (PB1)
- net LED2_2: now also U2.3 (PF1); no longer U2.17 (PA9)
- net LED2_3: now also R4.1, U2.17 (PA9), U3.6 (SCL); no longer R6.1, U2.18 (PA10)
- net LED3_1: now also U2.9 (PA3); no longer U2.11 (PA5)
- net LED3_2: now also R8.1, U2.8 (PA2); no longer R7.1, U2.3 (PF1)
- net LED3_3: now also R7.1, U2.7 (PA1); no longer R8.1, U2.2 (PF0)
- net PB1: now also PB1.2, U2.2 (PF0); no longer PB2.2, U2.12 (PA6)
- net PB2: now also PB2.2, U2.10 (PA4); no longer PB1.2, U2.13 (PA7)
- net RELE: now also U2.11 (PA5); no longer U2.10 (PA4)
- net RELE_LED1: now also R3.1, U2.14 (PB1); no longer R2.1, U2.6 (PA0)
- net RELE_LED2: now also R2.1, U2.13 (PA7); no longer R3.1, U2.7 (PA1)
- net SWDIO: now also J1.4 (Pin_4)
- net VDD: now also C4.1, C6.1, U1.3 (VI)
- net SENS1 renamed SDA
- net SDA: now also U2.18 (PA10), U3.5 (SDA); no longer U2.9 (PA3)
- removed net SENS2: J1.4 (Pin_4), U2.8 (PA2)
- new net: D1.4 (BA), R11.2
- new net RELE_LED3: R11.1, U2.12 (PA6)
Other:
- moved on the sheet: C1, C2, C3, D1, D2, D3, J1, J2, PB1, PB2, Q1, R1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

Commit message: пока без eeprom
Parts:
- removed U3: AT24CS64-SSHM, Package_SO:SO-8_5.3x6.2mm_P1.27mm, symbol Memory_EEPROM:AT24CS64-SSHM
- added PB3: Reset, кнопки:PB_SMD_3x6x2.5, symbol кнопки:кнопка
- C1: value C -> 0.1
- R1: value R -> 10k
- R11, R4, R7: value 64 -> 62
- R2, R5, R8: value 104 -> 100
- R3, R6, R9: value 224 -> 220
- U1: footprint Package_TO_SOT_SMD:SOT-223 -> Package_TO_SOT_SMD:SOT-223-3_TabPin2
Connections:
- net GNDD: now also PB3.2
- net at C1.2, R1.2, U2.4 (NRST): now also PB3.1
- net SDA renamed SENS1
Other:
- moved on the sheet: C2, C3, C4, C6, U1
