File: kicad/mcu/stm32f030f4p6/mcu.kicad_pcb (KiCad board)
At the start: 2 copper layers, 42.1 x 32.8 mm, 28 parts, among them J1 Conn_01x05, J2 Conn_01x04, Q1 BC817, U1 LM1117-3.3, U2 STM32F030F4P6

Commit message: Сенсоры перепутал-поправил. Усправил выход у Реле с OD на PP
Connections:
- net /SENS1 renamed /SENS2
Routing:
- net (no net): vias 4 -> 0
Changed lines of the file:
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@@
   (net 6 "/SWGCLK")
   (net 7 "Net-(D1-Pad4)")
-  (net 8 "/SENS1")
+  (net 8 "/SENS2")
   (net 9 "/RELE")
   (net 10 "/PB2")
@@
       (net 14 "/LED2_3") (pinfunction "PA9") (pintype "bidirectional"))
     (pad "18" smd roundrect (at 2.8625 1.625 180) (size 1.475 0.4) (layers "B.Cu" "B.Paste" "B.Mask") (roundrect_rratio 0.25)
-      (net 8 "/SENS1") (pinfunction "PA10") (pintype "bidirectional"))
+      (net 8 "/SENS2") (pinfunction "PA10") (pintype "bidirectional"))
     (pad "19" smd roundrect (at 2.8625 2.275 180) (size 1.475 0.4) (layers "B.Cu" "B.Paste" "B.Mask") (roundrect_rratio 0.25)
       (net 5 "/SWDIO") (pinfunction "PA13") (pintype "bidirectional"))
@@
       (net 28 "/RELE_OUT") (pinfunction "Pin_2") (pintype "passive"))
     (pad "3" thru_hole oval locked (at 5 0 90) (size 2 2.2) (drill 0.95) (layers *.Cu *.Mask)
-      (net 8 "/SENS1") (pinfunction "Pin_3") (pintype "passive"))
+      (net 8 "/SENS2") (pinfunction "Pin_3") (pintype "passive"))
     (pad "4" thru_hole oval locked (at 7.5 0 90) (size 2 2.2) (drill 0.95) (layers *.Cu *.Mask)
       (net 5 "/SWDIO") (pinfunction "Pin_4") (pintype "passive"))
@@
     (style (thickness 0.15) (arrow_length 1.27) (text_position_mode 0) (extension_height 0.58642) (extension_offset 0.5) keep_text_aligned)
   )
-  (via (at 270.09 15.24) (size 1.8) (drill 0.5) (layers "F.Cu" "B.Cu") (free) (net 0))
-  (via (at 270.09 54.61) (size 1.8) (drill 0.5) (layers "F.Cu" "B.Cu") (free) (net 0))
-  (via (at 221.83 54.61) (size 1.8) (drill 0.5) (layers "F.Cu" "B.Cu") (free) (net 0))
-  (via (at 221.83 15.24) (size 1.8) (drill 0.5) (layers "F.Cu" "B.Cu") (free) (net 0))
   (segment (start 228.388 27.872) (end 229.45 27.872) (width 0.8) (layer "F.Cu") (net 1))
   (segment (start 229.45 27.872) (end 230.398 26.924) (width 0.8) (layer "F.Cu") (net 1))

Commit message: Косметика
Parts:
- J2: value Conn_01x04 -> Conn_01x05; footprint Connector_JST:JST_EH_B4B-EH-A_1x04_P2.50mm_Vertical -> Connector_JST:JST_EH_B5B-EH-A_1x05_P2.50mm_Vertical
- moved J2 1.84 mm to (228.9, 23.6)
- moved C5 0.38 mm to (232.9, 24.9)
Connections:
- J2 pad 1: /SWDIO -> Net-(C1-Pad2)
- J2 pad 2: GNDD -> /SWDIO
- J2 pad 3: /SWGCLK -> GNDD
- J2 pad 4: VDD -> /SWGCLK
Routing:
- net Net-(C1-Pad2): track 15.4 -> 27.8 mm
- net /SWDIO: track 68.1 -> 66.8 mm
- net /SWGCLK: track 18.1 -> 19.0 mm
- net VDD: track 77.7 -> 76.9 mm
Other:
- board text added: "5V"
- board text added: "CLK"
- board text added: "GND"
- board text added: "IO"
- board text added: "RES"
- board text added: "SWD"
